File: hardware/src files/calve_heater/calve_heater.kicad_pcb (KiCad board)
At the start: 2 copper layers, 43.8 x 25 mm, 70 parts, among them J1 USB_B_Micro, J2 Conn_out, J3 ICSP_HEADER, Q1 FDN338P-NL, Q2 SI2304BDS-T1-GE3, SW1 SW_Push, SW2 SW_Push, U1 BQ24075RGT, U2 TPS61230DRCR, U3 ATmega328P-MU, U4 EAST1616RGBA8, U5 LM1117-3.3, Y1 X322516MOB4SI

Commit message: update on calve design
Parts:
- renumbered SW2 to PWR_BTN, SW1 to TEMP_BTN
